File: Marble_Tiny/Power.kicad_sch (KiCad schematic)
At the start: 63 parts, among them IC5 SN74LVC1G07DBV, IC6 SN74LVC1G07DBV, J10 Barrel_Jack_Switch, Q4 DMP3013SFV, U10 TPSM863257RDXR, U11 TPSM863257RDXR, U18 TLV77325PDBVR, U20 RT9045AGSP / AP2303, U4 TPSM863257RDXR, U5 TPSM863257RDXR, U6 TPSM863257RDXR

Commit message: components placement done, fixed issue with PCB
Parts:
- B5: footprint SON65P300X300X100-9N-D -> ICs And Semiconductors SMD:SON65P300X300X100-9N-R170X245
- U18: footprint DBV0005A_MFG -> Package_TO_SOT_SMD:SOT-23-5
- U20: footprint SOIC127P600X155-9N -> ICs And Semiconductors SMD:SOIC127P600X168-9N-S230
Changed lines of the file:
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@@
 (kicad_sch
-	(version 20241209)
+	(version 20250114)
 	(generator "eeschema")
 	(generator_version "9.0")
@@
 			)
 		)
-		(property "Footprint" "SOIC127P600X155-9N"
+		(property "Footprint" "ICs And Semiconductors SMD:SOIC127P600X168-9N-S230"
 			(at 228.6 93.98 0)
 			(effects
@@
 			)
 		)
-		(property "Footprint" "SON65P300X300X100-9N-D"
+		(property "Footprint" "ICs And Semiconductors SMD:SON65P300X300X100-9N-R170X245"
 			(at 212.09 118.11 0)
 			(effects
@@
 			)
 		)
-		(property "Footprint" "DBV0005A_MFG"
+		(property "Footprint" "Package_TO_SOT_SMD:SOT-23-5"
 			(at 210.82 144.78 0)
 			(effects
