File: Marble_Tiny/SFP.kicad_sch (KiCad schematic)
At the start: 73 parts, among them IC4 PCA9546ARGV, J1 TYCO_1888247-1, J11 TYCO_1888247-1, J12 TYCO_1888247-1, J13 TYCO_1888247-1, J8 2180739-1, J9 2180739-1, U17 TCA9535RTWR, U19 TCA9535RTWR

Commit message: components placement done, fixed issue with PCB
Parts:
- U17, U19: footprint RTW0024B_V -> ICs And Semiconductors SMD:QFN50P400X400X80-25N-S245
Changed lines of the file:
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@@
 (kicad_sch
-	(version 20241209)
+	(version 20250114)
 	(generator "eeschema")
 	(generator_version "9.0")
@@
 			)
 		)
-		(property "Footprint" "RTW0024B_V"
+		(property "Footprint" "ICs And Semiconductors SMD:QFN50P400X400X80-25N-S245"
 			(at 344.17 26.67 0)
 			(effects
@@
 			)
 		)
-		(property "Footprint" "RTW0024B_V"
+		(property "Footprint" "ICs And Semiconductors SMD:QFN50P400X400X80-25N-S245"
 			(at 344.17 95.25 0)
 			(effects
