File: Marble_Tiny/FPGA_PWR.kicad_sch (KiCad schematic)
At the start: 52 parts, among them U1 XC7A35T-CSG325

Commit message: fixed issue with PMODs; added board name and revision; fixed polygons issue
Other:
- company: (none) -> ${name}
Changed lines of the file:
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@@
 	(generator_version "9.0")
 	(paper "A4")
+	(title_block
+		(date "2025-04-18")
+		(rev "${rev}")
+		(company "${name}")
+		(comment 1 "${author}")
+	)
 	(junction
 		(at 203.2 124.46)
